File: blocks.kicad_blocks/LinearReg_XC6206P332MR-G.kicad_block/LinearReg_XC6206P332MR-G.kicad_pcb (KiCad board)
At the start: 2 copper layers, 6 parts, among them U1 XC6206P332MR-G

Commit message: nicer layout (#1)
* nicer layout

* fix: translate PR template to English, fix jlcpcb_basic field name

* fix: only flag README.md if it is new in the PR, not already on main

* fix: pr preview comment shows only changed blocks, not all
Parts:
- moved TP102 263.8 mm to (361.4, 78.2)
- moved C1 259.6 mm to (359.8, 73.2)
- moved U1 259.6 mm to (354.5, 79.5)
- moved C2 259.2 mm to (353.6, 74.2)
- moved C3 259.2 mm to (357.4, 74.2)
- moved TP103 258.7 mm to (358.1, 78.2)
Routing:
- net +5V: track 7.74 -> 4.59 mm
- net +3V3: track 16.8 -> 14.6 mm
- net GND: track 10.4 -> 12.2 mm, vias 6 -> 4
