File: blocks.kicad_blocks/USB-C_Socket_FullSpeed.kicad_block/USB-C_Socket_FullSpeed.kicad_sch (KiCad schematic)
At the start: 5 parts, among them J2 TYPE-C-31-M-12

Commit message: USB-C-Block: Footprint auf Projektbibliothek GnssFanout (KiCad-Std-Verweis war toter 3D-Pfad)
Parts:
- J2: footprint Connector_USB:USB_C_Receptacle_HRO_TYPE-C-31-M-12 -> GnssFanout:USB_C_Receptacle_HRO_TYPE-C-31-M-12
Changed lines of the file:
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@@
 			)
 		)
-		(property "Footprint" "Connector_USB:USB_C_Receptacle_HRO_TYPE-C-31-M-12"
+		(property "Footprint" "GnssFanout:USB_C_Receptacle_HRO_TYPE-C-31-M-12"
 			(at 697.23 163.98 0)
 			(hide yes)
